File: power-module/PM.kicad_sch (KiCad schematic)
At the start: 52 parts, among them J1 Conn_01x01, J2 Conn_01x04, J3 Conn_01x01, J4 Conn_01x16, U2 TAS5825MRHB

Commit message: wip
Parts:
- removed C26, C27, C28: 22n, Capacitor_SMD:C_0805_2012Metric, symbol Device:C
- removed FL3, FL4: PA2745NL, hw-footprints:PA2745NL, symbol Filter:Choke_Schaffner_RN102-0.3-02-12M
- added C36, C37, C38: 2n2, Capacitor_SMD:C_0603_1608Metric, symbol Device:C
- added FB1, FB2, FB3, FB4: 50R@100MHz, Inductor_SMD:L_1206_3216Metric, symbol Device:FerriteBead
- C33: value 22n -> 2n2; footprint Capacitor_SMD:C_0805_2012Metric -> Capacitor_SMD:C_0603_1608Metric; JLC C77069 -> C33353
- C7: JLC C48970670 -> C44606610
- C8: JLC C52994759 -> C44606610
- H1, H2, H3, H4: footprint MountingHole:MountingHole_3.2mm_M3_ISO14580_Pad -> MountingHole:MountingHole_2.7mm
Connections:
- net GND: now also C36.2, C37.2, C38.2
- net at C25.1, C4.1, C5.1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: now also FB3.1
- net at J2.4 (Pin_4): now also C36.1, FB1.2
- net at C1.1, C2.1, C3.1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: now also FB4.1
- net at J2.3 (Pin_3): now also C33.1, FB2.2
- net at C20.2, C22.2, C23.2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: now also FB1.1
- net at C17.2, C18.2, C19.2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: now also FB2.1
- net at J2.2 (Pin_2): now also C37.1, FB4.2; no longer C33.1
- net at J2.1 (Pin_1): now also C38.1, FB3.2

Commit message: WIP
TODO: Silk PM module. toslink module
Parts:
- added C26, C27: 22u, Capacitor_SMD:C_0805_2012Metric, symbol Device:C
Connections:
- net +24V: now also C26.1, C27.1
- net GND: now also C26.2, C27.2

Commit message: JLC MPN fixes, minor tweaks
Parts:
- J4: JLC C6120049 -> C5510131
Changed lines of the file:
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@@
 			)
 		)
-		(property "JLC" "C6120049"
+		(property "JLC" "C5510131"
 			(at 46.99 46.99 0)
 			(hide yes)
