File: streaming-module/streamer.kicad_sch (KiCad schematic)
At the start: 49 parts, among them J1 Conn_01x02, J2 Conn_01x04, J3 HS HS91L02W2C01, J4 Conn_01x15, J5 Conn_01x02, J6 Conn_02x13_Odd_Even, P1 USB_C_Plug_USB2.0, SW1 RotaryEncoder_Switch, U1 ESP32-S3-WROOM-1, U2 IRM-90-24, U4 SRV05-4, U6 TPS54202DDC, Y1 32k, Y2 22.5792M

Commit message: wip
Parts:
- removed J4: Conn_01x15, Connector_PinHeader_1.00mm:PinHeader_1x15_P1.00mm_Vertical, symbol Connector_Generic:Conn_01x15
- removed J6: Conn_02x13_Odd_Even, hw-footprints:GT-B0802 FSR 51-26, symbol Connector_Generic:Conn_02x13_Odd_Even
- added J7: Conn_01x16, hw-footprints:5034801600, symbol Connector_Generic:Conn_01x16
- added N1: amp board, symbol Mechanical:Housing
- J5: value Conn_01x02 -> AMP_PWR
Connections:
- net +24V: now also J5.2 (Pin_2), J7.5 (Pin_5)
- net +3V3: now also J7.1 (Pin_1)
- net AMP_IO1: now also J7.3 (Pin_3)
- net AMP_IO2: now also J7.4 (Pin_4)
- net AMP_~{PDN}: now also J7.15 (Pin_15)
- net GND: now also J7.11 (Pin_11), J7.13 (Pin_13), J7.16 (Pin_16), J7.2 (Pin_2), J7.6 (Pin_6), J7.8 (Pin_8)
- net LRCLK: now also J7.7 (Pin_7)
- net SCL: now also J7.14 (Pin_14)
- net SCLK: now also J7.9 (Pin_9)
- net SDA: now also J7.12 (Pin_12)
- net SDIN: now also J7.10 (Pin_10)

Commit message: WIP
Parts:
- removed FL1: Choke_CommonMode_PulseElectronics_PH9455x156NL, Inductor_THT:L_CommonMode_PulseElectronics_PH9455xxx6NL_2, symbol Filter:Choke_CommonMode_PulseElectronics_PH9455x156NL
- removed J1: Conn_01x02, symbol Connector_Generic:Conn_01x02
- removed J5: AMP_PWR, symbol Connector_Generic:Conn_01x02
- added C7: C_Polarized, Capacitor_THT:CP_Radial_D8.0mm_P3.50mm, symbol Device:C_Polarized
- added F1: Fuse, Fuse:Fuse_2512_6332Metric, symbol Device:Fuse
- added J4, J5: Conn_01x01, Connector_Wire:SolderWirePad_1x01_SMD_4x8mm, symbol Connector_Generic:Conn_01x01
- added J6, J8: Conn_01x01, Connector_Wire:SolderWire-1.5sqmm_1x01_D1.7mm_OD3mm, symbol Connector_Generic:Conn_01x01
- added R21: 8.2, Resistor_SMD:R_1206_3216Metric, symbol Device:R
- J7: footprint hw-footprints:5034801600 -> components:5034801600
- L5: footprint Inductor_SMD:L_APV_ANR5040 -> Inductor_SMD:L_APV_ANR6028; JLC C167967 -> C2849524
Connections:
- net +24V: now also C7.1, J4.1 (Pin_1), R21.2
- net GND: now also U2.4 (-Vout), C7.2, J5.1 (Pin_1)
- net at U2.1 (AC/L): now also F1.2
- net at U2.2 (AC/N): now also J8.1 (Pin_1)
- net at U2.3 (+Vout): now also R21.1
- new net: F1.1, J6.1 (Pin_1)

Commit message: wip
Parts:
- removed C6: 100n, Capacitor_SMD:C_0402_1005Metric, symbol Device:C
- removed R15: 22, Resistor_SMD:R_0402_1005Metric, symbol Device:R
- removed R8: 4k7, Resistor_SMD:R_0402_1005Metric, symbol Device:R
- removed Y2: 22.5792M, Crystal:Crystal_SMD_3225-4Pin_3.2x2.5mm, symbol Oscillator:SiT8008xx-1x-xxE
- F1: JLC (none) -> C2762422
- J4: value Conn_01x01 -> AMP_24V
- J5: value Conn_01x01 -> AMP_GND
- N1: footprint (none) -> components:virtual_component
Connections:
- net +24V: no longer C7.1, J4.1 (Pin_1), R21.2
- net AMP_~{PDN}: now also U1.31 (IO38)
- net CC1: now also U4.4 (IO3); no longer U4.6 (IO4)
- net CC2: now also U4.6 (IO4); no longer U4.4 (IO3)
- net GND: no longer C7.2, J5.1 (Pin_1), U2.4 (-Vout)
- net CLK_EN: no longer names the net of U1.15 (IO3)
- net I2S_MCLK: no longer names the net of U1.7 (IO7)
- new net: C7.1, J4.1 (Pin_1), R21.2
- new net GNDPWR: C7.2, J5.1 (Pin_1), U2.4 (-Vout)
Other:
- moved on the sheet: J4, J5, N1

Commit message: WIP
Parts:
- removed R21: 8.2, Resistor_SMD:R_1206_3216Metric, symbol Device:R
- added C10: 22u 6.3V, Capacitor_SMD:C_0805_2012Metric, symbol Device:C
- added C11, C12, C13, C14, C15, C16: 100n, Capacitor_SMD:C_0402_1005Metric, symbol Device:C
- added C6: 4n7, Capacitor_SMD:C_0603_1608Metric, symbol Device:C
- added C8: 68n, Capacitor_SMD:C_1206_3216Metric, symbol Device:C
- added FB5: 50R@100MHz, Inductor_SMD:L_1206_3216Metric, symbol Device:FerriteBead
- added R2: 680, Resistor_SMD:R_0402_1005Metric, symbol Device:R
- added R22: 22k, Resistor_SMD:R_0402_1005Metric, symbol Device:R
- added R23, R24, R25, R26, R27, R28, R29, R30, R31: 22, Resistor_SMD:R_0402_1005Metric, symbol Device:R
- added R3, R4, R8: 0, Resistor_SMD:R_0402_1005Metric, symbol Device:R
- added TP1: BFRAME, TestPoint:TestPoint_Pad_2.0x2.0mm, symbol Connector:TestPoint
- added TP2: UOUT, TestPoint:TestPoint_Pad_2.0x2.0mm, symbol Connector:TestPoint
- added TP3: COUT, TestPoint:TestPoint_Pad_2.0x2.0mm, symbol Connector:TestPoint
- added U3: DIR9001PWR, easyeda2kicad:TSSOP-28_L9.7-W4.4-P0.65-LS6.4-BL, symbol easyeda2kicad:DIR9001PWR
- added U5, U7, U8: TP74LVC1G157C6, Package_TO_SOT_SMD:SOT-363_SC-70-6, symbol Analog_Switch:FSA3157P6X
- added U9: PM2.54-1*3, easyeda2kicad:HDR-TH_3P-P2.54-V-F, symbol easyeda2kicad:PM2.54-1*3
- J4, J5: footprint Connector_Wire:SolderWirePad_1x01_SMD_4x8mm -> Connector_Wire:SolderWire-2.5sqmm_1x01_D2.4mm_OD3.6mm
- P1: footprint Connector_USB:USB_C_Receptacle_HCTL_HC-TYPE-C-16P-01A -> components:MC-710S-Z13
Connections:
- net +3V3: now also C10.1, C11.1, C13.1, C14.1, C15.1, C16.1, R22.1, U3.24 (VCC), U3.25 (FMT0), U3.26 (FMT1), U3.5 (VDD), U5.5 (V+), U7.5 (V+), U8.5 (V+), U9.1
- net CC1: now also U4.6 (IO4); no longer U4.4 (IO3)
- net CC2: now also U4.4 (IO3); no longer U4.6 (IO4)
- net D+: now also U4.3 (IO2)
- net D-: now also U4.1 (IO1)
- net GND: now also C10.2, C11.2, C12.2, C13.2, C14.2, C15.2, C16.2, C6.1, C8.1, U3.13 (PSCK0), U3.14 (PSCK1), U3.19 (RSV), U3.23 (AGND), U3.28 (CKSEL), U3.6 (DGND), U3.8 (XTI), U5.2 (GND), U7.2 (GND), U8.2 (GND), U9.3
- net LRCLK: now also R30.2, R4.2; no longer U1.34 (IO41)
- net SCLK: now also R31.2, R8.2; no longer U1.35 (IO42)
- net SDIN: now also R29.2, R3.2; no longer U1.26 (IO45)
- net at U2.3 (+Vout): now also FB5.1
- net at P1.A7 (D-), P1.B7 (D-), R16.1: no longer U4.1 (IO1)
- net at P1.A6 (D+), P1.B6 (D+), R17.1: no longer U4.3 (IO2)
- net at C7.1, J4.1 (Pin_1): now also FB5.2
- net I2S_MUX: now reaches U1.20 (IO12)
- net I2S_MUX: now also U5.6, U7.6, U8.6
- net OPT_~{CLK_OK}: now reaches U1.21 (IO13)
- net OPT_~{CLK_OK}: now also U3.27 (ERROR)
- net OPT_~{AUDIO}: now reaches U1.22 (IO14)
- net OPT_~{AUDIO}: now also U3.1 (~{AUDIO})
- new net: C6.2, R2.1, U3.22 (FILT)
- new net: C8.2, R2.2
- new net: R27.2, U3.11 (BCKO)
- new net: R28.2, U3.12 (DOUT)
- new net: TP2.1, U3.16 (UOUT)
- new net: R25.1, U1.26 (IO45)
- new net: R26.2, U3.10 (LRCKO)
- new net: R29.1, U7.4
- new net: TP3.1, U3.15 (COUT)
- new net: TP1.1, U3.18 (BFRAME)
- new net: R31.1, U5.4
- new net: R30.1, U8.4
- new net: R24.1, U1.35 (IO42)
- new net: R23.1, U1.34 (IO41)
- new net ESP_LRCLK: R23.2, R4.1, U8.3
- new net ESP_SCLK: R24.2, R8.1, U5.3
- new net ESP_SDOUT: R25.2, R3.1, U7.3
- new net OPT_LRCLK: R26.1, U8.1
- new net OPT_SCLK: R27.1, U5.1
- new net OPT_SDOUT: R28.1, U7.1
- new net OPT_~{RST}: C12.1, R22.2, U3.21 (~{RST})
- new net TOSLINK_IN: U3.20 (RXIN), U9.2
- no-connect marks 0 -> 5
Other:
- note added: "AC-DC"
- note added: "DC-DC"
- note added: "ESP32"
- note added: "Optical input"
- note added: "USB"
- note added: "remove if adding opt input"
- moved on the sheet: C1, C2, C22, C23, C24, C25, C26, C27, C28, C3, C33, C4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

Commit message: WIP
TODO: Silk PM module. toslink module
Parts:
- P1: footprint components:MC-710S-Z13 -> easyeda2kicad:USB-C-SMD_GT-USB-7058
Connections:
- net D+: now also R16.1; no longer R17.2, U4.3 (IO2)
- net D-: now also R17.1; no longer R16.2, U4.1 (IO1)
- net at P1.A6 (D+), P1.B6 (D+): now also R16.2, U4.3 (IO2); no longer R17.1
- net at P1.A7 (D-), P1.B7 (D-): now also R17.2, U4.1 (IO1); no longer R16.1
Other:
- moved on the sheet: R16, R17
Changed lines of the file:
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@@
 	)
 	(junction
+		(at 72.39 162.56)
+		(diameter 0)
+		(color 0 0 0 0)
+	)
+	(junction
 		(at 153.67 140.97)
 		(diameter 0)
@@
 	)
 	(junction
-		(at 72.39 162.56)
-		(diameter 0)
-		(color 0 0 0 0)
-	)
-	(junction
 		(at 60.96 95.25)
 		(diameter 0)
@@
 	)
 	(junction
-		(at 69.85 167.64)
-		(diameter 0)
-		(color 0 0 0 0)
-	)
-	(junction
 		(at 259.08 243.84)
 		(diameter 0)
@@
 	)
 	(junction
+		(at 67.31 167.64)
+		(diameter 0)
+		(color 0 0 0 0)
+	)
+	(junction
 		(at 99.06 95.25)
 		(diameter 0)
@@
 	(wire
 		(pts
-			(xy 69.85 167.64) (xy 69.85 173.99)
-		)
-		(stroke
-			(width 0)
-			(type default)
-		)
-	)
-	(wire
-		(pts
 			(xy 38.1 224.79) (xy 50.8 224.79)
 		)
@@
 	(wire
 		(pts
+			(xy 72.39 162.56) (xy 72.39 172.72)
+		)
+		(stroke
+			(width 0)
+			(type default)
+		)
+	)
+	(wire
+		(pts
 			(xy 382.27 154.94) (xy 378.46 154.94)
 		)
@@
 	(wire
 		(pts
-			(xy 45.72 167.64) (xy 46.99 167.64)
+			(xy 72.39 162.56) (xy 73.66 162.56)
 		)
 		(stroke
@@
 	(wire
 		(pts
-			(xy 245.11 165.1) (xy 245.11 166.37)
+			(xy 45.72 167.64) (xy 46.99 167.64)
 		)
 		(stroke
@@
 	(wire
 		(pts
-			(xy 45.72 162.56) (xy 58.42 162.56)
+			(xy 245.11 165.1) (xy 245.11 166.37)
 		)
 		(stroke
@@
 	(wire
 		(pts
-			(xy 233.68 96.52) (xy 236.22 96.52)
+			(xy 45.72 162.56) (xy 72.39 162.56)
 		)
 		(stroke
@@
 	(wire
 		(pts
-			(xy 153.67 66.04) (xy 163.83 66.04)
+			(xy 233.68 96.52) (xy 236.22 96.52)
 		)
 		(stroke
@@
 	(wire
 		(pts
-			(xy 66.04 167.64) (xy 69.85 167.64)
+			(xy 153.67 66.04) (xy 163.83 66.04)
 		)
 		(stroke
@@
 	(wire
 		(pts
+			(xy 67.31 182.88) (xy 67.31 180.34)
+		)
+		(stroke
+			(width 0)
+			(type default)
+		)
+	)
+	(wire
+		(pts
 			(xy 175.26 161.29) (xy 173.99 161.29)
 		)
@@
 	(wire
 		(pts
+			(xy 72.39 180.34) (xy 72.39 182.88)
+		)
+		(stroke
+			(width 0)
+			(type default)
+		)
+	)
+	(wire
+		(pts
 			(xy 199.39 264.16) (xy 195.58 264.16)
 		)
@@
 	(wire
 		(pts
+			(xy 67.31 167.64) (xy 67.31 172.72)
+		)
+		(stroke
+			(width 0)
+			(type default)
+		)
+	)
+	(wire
+		(pts
 			(xy 200.66 156.21) (xy 204.47 156.21)
 		)
@@
 	(wire
 		(pts
+			(xy 67.31 167.64) (xy 73.66 167.64)
+		)
+		(stroke
+			(width 0)
+			(type default)
+		)
+	)
+	(wire
+		(pts
 			(xy 179.07 149.86) (xy 179.07 156.21)
 		)
@@
 	(wire
 		(pts
-			(xy 72.39 173.99) (xy 72.39 162.56)
-		)
-		(stroke
-			(width 0)
-			(type default)
-		)
-	)
-	(wire
-		(pts
 			(xy 22.86 187.96) (xy 22.86 189.23)
 		)
@@
 	(wire
 		(pts
-			(xy 69.85 167.64) (xy 73.66 167.64)
-		)
-		(stroke
-			(width 0)
-			(type default)
-		)
-	)
-	(wire
-		(pts
 			(xy 203.2 153.67) (xy 204.47 153.67)
 		)
@@
 	(wire
 		(pts
-			(xy 46.99 167.64) (xy 58.42 167.64)
+			(xy 46.99 167.64) (xy 67.31 167.64)
 		)
 		(stroke
@@
 	(wire
 		(pts
-			(xy 66.04 162.56) (xy 72.39 162.56)
-		)
-		(stroke
-			(width 0)
-			(type default)
-		)
-	)
-	(wire
-		(pts
 			(xy 66.04 269.24) (xy 67.31 269.24)
 		)
@@
 	(wire
 		(pts
-			(xy 72.39 162.56) (xy 73.66 162.56)
-		)
-		(stroke
-			(width 0)
-			(type default)
-		)
-	)
-	(wire
-		(pts
 			(xy 256.54 55.88) (xy 257.81 55.88)
 		)
@@
 	)
 	(label "D+"
-		(at 69.85 173.99 270)
+		(at 67.31 182.88 270)
 		(effects
 			(font
@@
 	)
 	(label "D-"
-		(at 72.39 173.99 270)
+		(at 72.39 182.88 270)
 		(effects
 			(font
@@
 	(symbol
 		(lib_id "Device:R")
-		(at 62.23 167.64 90)
+		(at 72.39 176.53 180)
 		(unit 1)
 		(body_style 1)
@@
 		(dnp no)
 		(property "Reference" "R17"
-			(at 62.484 169.926 90)
+			(at 74.676 176.276 90)
 			(show_name no)
 			(do_not_autoplace no)
@@
 		)
 		(property "Value" "22"
-			(at 62.23 167.64 90)
+			(at 72.39 176.53 90)
 			(show_name no)
 			(do_not_autoplace no)
@@
 		)
 		(property "Footprint" "Resistor_SMD:R_0402_1005Metric"
-			(at 62.23 169.418 90)
+			(at 74.168 176.53 90)
 			(hide yes)
 			(show_name no)
@@
 		)
 		(property "Datasheet" ""
-			(at 62.23 167.64 0)
+			(at 72.39 176.53 0)
 			(hide yes)
 			(show_name no)
@@
 		)
 		(property "Description" "Resistor"
-			(at 62.23 167.64 0)
+			(at 72.39 176.53 0)
 			(hide yes)
 			(show_name no)
@@
 		)
 		(property "JLC" "C25092"
-			(at 62.23 167.64 90)
+			(at 72.39 176.53 90)
 			(hide yes)
 			(show_name no)
@@
 		)
 		(property "Voltage rating" ""
-			(at 62.23 167.64 90)
+			(at 72.39 176.53 90)
 			(hide yes)
 			(show_name no)
@@
 			)
 		)
-		(property "Footprint" "components:MC-710S-Z13"
+		(property "Footprint" "easyeda2kicad:USB-C-SMD_GT-USB-7058"
 			(at 34.29 165.1 0)
 			(hide yes)
@@
 	(symbol
 		(lib_id "Device:R")
-		(at 62.23 162.56 90)
+		(at 67.31 176.53 180)
 		(unit 1)
 		(body_style 1)
@@
 		(dnp no)
 		(property "Reference" "R16"
-			(at 62.484 160.02 90)
+			(at 64.77 176.276 90)
 			(show_name no)
 			(do_not_autoplace no)
@@
 		)
 		(property "Value" "22"
-			(at 62.23 162.56 90)
+			(at 67.31 176.53 90)
 			(show_name no)
 			(do_not_autoplace no)
@@
 		)
 		(property "Footprint" "Resistor_SMD:R_0402_1005Metric"
-			(at 62.23 164.338 90)
+			(at 69.088 176.53 90)
 			(hide yes)
 			(show_name no)
@@
 		)
 		(property "Datasheet" ""
-			(at 62.23 162.56 0)
+			(at 67.31 176.53 0)
 			(hide yes)
 			(show_name no)
@@
 		)
 		(property "Description" "Resistor"
-			(at 62.23 162.56 0)
+			(at 67.31 176.53 0)
 			(hide yes)
 			(show_name no)
@@
 		)
 		(property "JLC" "C25092"
-			(at 62.23 162.56 90)
+			(at 67.31 176.53 90)
 			(hide yes)
 			(show_name no)
@@
 		)
 		(property "Voltage rating" ""
-			(at 62.23 162.56 90)
+			(at 67.31 176.53 90)
 			(hide yes)
 			(show_name no)

Commit message: RFM
Parts:
- C6, C8, R2, U3, U5, U8, U9: now left out of the parts list
Changed lines of the file:
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@@
 		(body_style 1)
 		(exclude_from_sim no)
-		(in_bom yes)
+		(in_bom no)
 		(on_board yes)
 		(in_pos_files yes)
@@
 		(body_style 1)
 		(exclude_from_sim no)
-		(in_bom yes)
+		(in_bom no)
 		(on_board yes)
 		(in_pos_files yes)
@@
 		(unit 2)
 		(body_style 1)
-		(exclude_from_sim no)
+		(exclude_from_sim yes)
 		(in_bom yes)
 		(on_board yes)
@@
 		(body_style 1)
 		(exclude_from_sim no)
-		(in_bom yes)
+		(in_bom no)
 		(on_board yes)
 		(in_pos_files yes)
@@
 		(body_style 1)
 		(exclude_from_sim no)
-		(in_bom yes)
+		(in_bom no)
 		(on_board yes)
 		(in_pos_files yes)
@@
 		(body_style 1)
 		(exclude_from_sim no)
-		(in_bom yes)
+		(in_bom no)
 		(on_board yes)
 		(in_pos_files yes)
@@
 		(body_style 1)
 		(exclude_from_sim no)
-		(in_bom yes)
+		(in_bom no)
 		(on_board yes)
 		(in_pos_files yes)
@@
 		(body_style 1)
 		(exclude_from_sim no)
-		(in_bom yes)
+		(in_bom no)
 		(on_board yes)
 		(in_pos_files yes)
@@
 		(body_style 1)
 		(exclude_from_sim no)
-		(in_bom yes)
+		(in_bom no)
 		(on_board yes)
 		(in_pos_files yes)
@@
 		(body_style 1)
 		(exclude_from_sim no)
-		(in_bom yes)
+		(in_bom no)
 		(on_board yes)
 		(in_pos_files yes)

Commit message: JLC MPN fixes, minor tweaks
Parts:
- J7: JLC C6120049 -> C5510131
Changed lines of the file:
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@@
 			)
 		)
-		(property "JLC" "C6120049"
+		(property "JLC" "C5510131"
 			(at 387.35 165.1 0)
 			(hide yes)
